File: pcb/PCB remote.kicad_sch (KiCad schematic)
At the start: 11 parts, among them J1 Conn_01x01, J2 Conn_01x01, SW1 GREEN, SW2 RED, U1 RFM69HW, U2 SSD1306, U3 Joystick

Commit message: Update PCB design with latest changes
Parts:
- U1: footprint RF_Module:HOPERF_RFM69HW -> Remote-footprints:RFM69HCW(homemade)
Changed lines of the file:
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@@
 			)
 		)
-		(property "Footprint" "RF_Module:HOPERF_RFM69HW"
+		(property "Footprint" "Remote-footprints:RFM69HCW(homemade)"
 			(at 86.36 64.77 0)
 			(effects

Commit message: ny pcb og noget nyt code glete at gemme de andre dage men her er et push
Parts:
- added C4: 10uF, Capacitor_SMD:C_0805_2012Metric_Pad1.18x1.45mm_HandSolder, symbol Device:C
- added J3: 02_Socket, Connector_JST:JST_PH_S2B-PH-K_1x02_P2.00mm_Horizontal, symbol Connector:Conn_01x02_Socket
- added J4: Conn_01x02_Socket, Connector_Wire:SolderWire-0.5sqmm_1x02_P4.8mm_D0.9mm_OD2.3mm, symbol Connector:Conn_01x02_Socket
- added Q1: PMV28XPEAR, Remote-footprints:Pmos, symbol Remote-PCB-dele:PMV28XPEAR
- added Q2: BSS138, Remote-footprints:nmos, symbol Remote-PCB-dele:BSS138
- added R1: 220k, Resistor_SMD:R_0805_2012Metric_Pad1.20x1.40mm_HandSolder, symbol Device:R
- added R2: 47k, Resistor_SMD:R_0603_1608Metric_Pad0.98x0.95mm_HandSolder, symbol Device:R
- added S1: 100SP1T1B1M7QEH, Remote-footprints:100SP1T1B1M7QEH(redSwitch), symbol Remote-PCB-dele:100SP1T1B1M7QEH
- added U4: HW373, Remote-footprints:HW373, symbol Remote-PCB-dele:HW373
- C1: value 10u -> 10uF
- C2, C3: value 100n -> 100nF
Connections:
- net GND: now also C4.2, J4.1 (Pin_1), J4.2 (Pin_2), Q2.2 (S), R2.2, U4.4 (out-)
- net PWRControl: now reaches A1.19 (D5)
- net PWRControl: now also Q2.1 (G), R2.1
- net +BATT: now reaches A1.28 (VBAT)
- net +BATT: now also Q1.3 (D)
- new net: C4.1, Q1.1 (G), Q2.3 (D), R1.2
- new net: J3.1 (Pin_1), U4.2 (b-)
- new net: J3.2 (Pin_2), U4.1 (b+)
- new net: S1.2 (COM), U4.3 (out+)
- new net: Q1.2 (S), R1.1, S1.3 (NO)
Other:
- note added: "Battery control"
- note added: "Main system"
- moved on the sheet: A1, C1, C2, C3, J1, J2, SW1, SW2, U1
